File: esc.sch (KiCad schematic (older format))
At the start: 26 parts, among them IC1 4N25, IC2 ATMEGA8-AI, P1 CONN_01X03, P2 CONN_01X02, P3 CONN_01X03, U1 LM2931AZ-5.0

Commit message: Added PWR flag
Connections:
- net labels removed: PWM_to_atmel
- wire segments 28 -> 30
Other:
- moved on the sheet: P2, Q?, R?
Changed lines of the file:
@@
 L CONN_01X02 P2
 U 1 1 564456C5
-P 950 2000
-F 0 "P2" H 950 2150 50  0000 C CNN
-F 1 "CONN_01X02" V 1050 2000 50  0000 C CNN
-F 2 "" H 950 2000 60  0000 C CNN
-F 3 "" H 950 2000 60  0000 C CNN
-	1    950  2000
+P 850 2000
+F 0 "P2" H 850 2150 50  0000 C CNN
+F 1 "CONN_01X02" V 950 2000 50  0000 C CNN
+F 2 "" H 850 2000 60  0000 C CNN
+F 3 "" H 850 2000 60  0000 C CNN
+	1    850  2000
 	-1   0    0    1
 $EndComp
@@
 Text GLabel 1150 1950 2    60   Output ~ 0
 V_BAT
-Text Notes 900  1750 0    60   ~ 0
+Text Notes 800  1750 0    60   ~ 0
 BAT
 $Comp
@@
 PWM
 Connection ~ 4600 8200
-Text Label 4600 8000 0    60   ~ 0
-PWM_to_atmel
 Text GLabel 4400 8600 2    60   Input ~ 0
 M
@@
 L MOSFET_N Q?
 U 1 1 5645A4E6
-P 13050 2850
-F 0 "Q?" H 13060 3020 60  0000 R CNN
-F 1 "MOSFET_N" H 13060 2700 60  0000 R CNN
-F 2 "" H 13050 2850 60  0000 C CNN
-F 3 "" H 13050 2850 60  0000 C CNN
-	1    13050 2850
+P 14150 2750
+F 0 "Q?" H 14160 2920 60  0000 R CNN
+F 1 "MOSFET_N" H 14160 2600 60  0000 R CNN
+F 2 "" H 14150 2750 60  0000 C CNN
+F 3 "" H 14150 2750 60  0000 C CNN
+	1    14150 2750
 	1    0    0    -1
 $EndComp
@@
 L MOSFET_P Q?
 U 1 1 5645A545
-P 13050 2250
-F 0 "Q?" H 13050 2440 60  0000 R CNN
-F 1 "MOSFET_P" H 13050 2070 60  0000 R CNN
-F 2 "" H 13050 2250 60  0000 C CNN
-F 3 "" H 13050 2250 60  0000 C CNN
-	1    13050 2250
+P 14150 2150
+F 0 "Q?" H 14150 2340 60  0000 R CNN
+F 1 "MOSFET_P" H 14150 1970 60  0000 R CNN
+F 2 "" H 14150 2150 60  0000 C CNN
+F 3 "" H 14150 2150 60  0000 C CNN
+	1    14150 2150
 	1    0    0    1
 $EndComp
-Text GLabel 13600 2550 2    60   Output ~ 0
+Text GLabel 14700 2450 2    60   Output ~ 0
 A
 Wire Wire Line
-	13150 2450 13150 2650
-Wire Wire Line
-	10350 2550 13600 2550
-Connection ~ 13150 2550
+	14250 2350 14250 2550
+Wire Wire Line
+	11450 2450 14700 2450
+Connection ~ 14250 2450
 $Comp
 L R R?
 U 1 1 5645B08B
-P 10100 2550
-F 0 "R?" V 10180 2550 40  0000 C CNN
-F 1 "18k" V 10107 2551 40  0000 C CNN
-F 2 "" V 10030 2550 30  0000 C CNN
-F 3 "" H 10100 2550 30  0000 C CNN
-	1    10100 2550
+P 11200 2450
+F 0 "R?" V 11280 2450 40  0000 C CNN
+F 1 "18k" V 11207 2451 40  0000 C CNN
+F 2 "" V 11130 2450 30  0000 C CNN
+F 3 "" H 11200 2450 30  0000 C CNN
+	1    11200 2450
 	0    1    1    0
 $EndComp
@@
 L R R?
 U 1 1 5645B23F
-P 9750 3100
-F 0 "R?" V 9830 3100 40  0000 C CNN
-F 1 "3k3" V 9757 3101 40  0000 C CNN
-F 2 "" V 9680 3100 30  0000 C CNN
-F 3 "" H 9750 3100 30  0000 C CNN
-	1    9750 3100
+P 10850 3000
+F 0 "R?" V 10930 3000 40  0000 C CNN
+F 1 "3k3" V 10857 3001 40  0000 C CNN
+F 2 "" V 10780 3000 30  0000 C CNN
+F 3 "" H 10850 3000 30  0000 C CNN
+	1    10850 3000
 	1    0    0    -1
 $EndComp
@@
 L R R?
 U 1 1 5645B3A7
-P 9400 2550
-F 0 "R?" V 9480 2550 40  0000 C CNN
-F 1 "3k3" V 9407 2551 40  0000 C CNN
-F 2 "" V 9330 2550 30  0000 C CNN
-F 3 "" H 9400 2550 30  0000 C CNN
-	1    9400 2550
-	0    1    1    0
-$EndComp
-Text GLabel 9150 2550 0    60   Output ~ 0
+P 10500 2450
+F 0 "R?" V 10580 2450 40  0000 C CNN
+F 1 "3k3" V 10507 2451 40  0000 C CNN
+F 2 "" V 10430 2450 30  0000 C CNN
+F 3 "" H 10500 2450 30  0000 C CNN
+	1    10500 2450
+	0    1    1    0
+$EndComp
+Text GLabel 10250 2450 0    60   Output ~ 0
 M
 $Comp
 L GND #PWR?
 U 1 1 5645BC30
-P 9750 3350
-F 0 "#PWR?" H 9750 3350 30  0001 C CNN
-F 1 "GND" H 9750 3280 30  0001 C CNN
-F 2 "" H 9750 3350 60  0000 C CNN
-F 3 "" H 9750 3350 60  0000 C CNN
-	1    9750 3350
-	1    0    0    -1
-$EndComp
-Text GLabel 9650 2750 0    60   Output ~ 0
+P 10850 3250
+F 0 "#PWR?" H 10850 3250 30  0001 C CNN
+F 1 "GND" H 10850 3180 30  0001 C CNN
+F 2 "" H 10850 3250 60  0000 C CNN
+F 3 "" H 10850 3250 60  0000 C CNN
+	1    10850 3250
+	1    0    0    -1
+$EndComp
+Text GLabel 10750 2650 0    60   Output ~ 0
 S_A
 Wire Wire Line
-	9650 2550 9850 2550
-Wire Wire Line
-	9750 2850 9750 2550
-Connection ~ 9750 2550
-Wire Wire Line
-	9650 2750 9750 2750
-Connection ~ 9750 2750
-Text GLabel 13150 2050 1    60   Input ~ 0
+	10750 2450 10950 2450
+Wire Wire Line
+	10850 2750 10850 2450
+Connection ~ 10850 2450
+Wire Wire Line
+	10750 2650 10850 2650
+Connection ~ 10850 2650
+Text GLabel 14250 1950 1    60   Input ~ 0
 V_BAT
 $Comp
 L GND #PWR?
 U 1 1 5645DA84
-P 13150 3050
-F 0 "#PWR?" H 13150 3050 30  0001 C CNN
-F 1 "GND" H 13150 2980 30  0001 C CNN
-F 2 "" H 13150 3050 60  0000 C CNN
-F 3 "" H 13150 3050 60  0000 C CNN
-	1    13150 3050
-	1    0    0    -1
-$EndComp
+P 14250 2950
+F 0 "#PWR?" H 14250 2950 30  0001 C CNN
+F 1 "GND" H 14250 2880 30  0001 C CNN
+F 2 "" H 14250 2950 60  0000 C CNN
+F 3 "" H 14250 2950 60  0000 C CNN
+	1    14250 2950
+	1    0    0    -1
+$EndComp
+$Comp
+L PWR_FLAG #FLG?
+U 1 1 5645F4FC
+P 1100 1950
+F 0 "#FLG?" H 1100 2045 30  0001 C CNN
+F 1 "PWR_FLAG" H 1100 2130 30  0000 C CNN
+F 2 "" H 1100 1950 60  0000 C CNN
+F 3 "" H 1100 1950 60  0000 C CNN
+	1    1100 1950
+	1    0    0    -1
+$EndComp
+$Comp
+L PWR_FLAG #FLG?
+U 1 1 5645F528
+P 1100 2050
+F 0 "#FLG?" H 1100 2145 30  0001 C CNN
+F 1 "PWR_FLAG" H 1100 2230 30  0000 C CNN
+F 2 "" H 1100 2050 60  0000 C CNN
+F 3 "" H 1100 2050 60  0000 C CNN
+	1    1100 2050
+	-1   0    0    1
+$EndComp
+Wire Wire Line
+	1050 2050 1150 2050
+Connection ~ 1100 2050
+Wire Wire Line
+	1050 1950 1150 1950
+Connection ~ 1100 1950
 $EndSCHEMATC

Commit message: Plan quasi fertig
Parts:
- removed Q?: MOSFET_P, symbol MOSFET_P
- added C1, C11, C2, C6, C8, C9: 1µ, symbol CP2
- added IC2, IC3, IC4: LM25101, symbol LM25101
- added Q1, Q10, Q11, Q12, Q2, Q3, Q5, Q6, Q7, Q8, Q9: MOSFET_N, symbol MOSFET_N
- added R10: 0 Bridge, symbol R
- added R11, R13, R15, R8: 3k3, symbol R
- added R14, R9: 18k, symbol R
- R6: renamed from R3; value R -> 1
- U1: value LM2931AZ-5.0 -> MCP1804; footprint TO92-123 -> ~
- gave numbers to parts that had none: 4
- renumbered C6 to C10, C3 to C12, C2 to C13, C8 to C14, C9 to C15, C10 to C16, C1 to C3, C7 to C5, C5 to C7, IC2 to IC5, P3 to P2, P2 to P3, R2 to R1, R1 to R12, R4 to R2, R5 to R7
Connections:
- net labels added: 9V
- wire segments 30 -> 71
Other:
- moved on the sheet: C10, C12, C13, C14, C15, C16, IC5, Q4, R12, R3, R4, R5

Commit message: Layout done!
Parts:
- removed R10: 0 Bridge, symbol R
- added C?: 22µ, symbol C
- added C?: 470n, symbol C
- added D1: DIODE, symbol DIODE
- added P?: CONN_02X02, symbol CONN_02X02
- added R16: 3k3, symbol R
- added R17: 0 Bridge, symbol R
- added U?: LM2940 10V, ~, symbol LM2931AZ-5.0
- added Y1: RESONATEUR, symbol RESONATEUR
Connections:
- net +5V: now also R16.2
- net 9V: now also C?.1, P?.2 (P2), U?.1 (VO)
- net GND: now also C?.2, C?.2, R17.2, U?.2 (GND), Y1.2; no longer IC5.14 ((~SS~/OC1B)PB2)
- net V_BAT: now also D1.1 (A), P?.1 (P1), P?.3 (P3); no longer R6.2
- net at IC5.7 (PB6(XTAL1/TOSC1)): now also Y1.1
- net at IC5.8 (PB7(XTAL2/TOSC2)): now also Y1.3
- net A_Lowside_Gate: now reaches IC2.8 (LO), Q3.G, Q4.G
- net A_Highside_Gate: now reaches IC2.3 (HO), Q1.G, Q2.G
- net B_Lowside_Gate: now reaches IC3.8 (LO), Q7.G, Q8.G
- net B_Highside_Gate: now reaches IC3.3 (HO), Q5.G, Q6.G
- net C_Lowside_Gate: now reaches IC4.8 (LO), Q11.G, Q12.G
- net C_Highside_Gate: now reaches IC4.3 (HO), Q10.G, Q9.G
- net MISO: no longer names the net of IC5.16 ((MISO)PB4)
- net MOSI: no longer names the net of IC5.15 ((MOSI/OC2)PB3)
- net RESET: no longer names the net of IC5.29 (PC6(~RESET~))
- net RESET: now also R16.1
- net SCK: no longer names the net of IC5.17 ((SCK)PB5)
- new net: IC5.14 ((~SS~/OC1B)PB2), R17.1
- new net: D1.2 (K), R6.2
- new net VBat_to_10V: C?.1, P?.4 (P4), U?.3 (VI)
- no-connect marks 7 -> 10
Other:
- note added: "ATMEGA8\n"
- note added: "H-Bridge Phase A"
- note added: "H-Bridge Phase B"
- note added: "H-Bridge Phase C"
- note added: "INPUT/OUTPUT"
- note added: "Optional"
- note added: "Switch: IF VBat < 14:\nBridge UP\n"
- note added: "VBat to 5V"
- note added: "VBat to 9-14V"
- moved on the sheet: C3

Commit message: Platiene begonnen
Parts:
- C1, C10, C11, C12, C13, C14, C15, C16, C2, C4, C5, C6, C7, C8, C9: footprint (none) -> Capacitors_SMD:C_0805_HandSoldering
- C17: renamed from C?; footprint (none) -> Capacitors_SMD:C_0805_HandSoldering
- C18: renamed from C?; footprint (none) -> Capacitors_SMD:C_1206
- C3: footprint (none) -> Capacitors_Elko_ThroughHole:Elko_vert_11x5mm_RM2_CopperClear
- D1: footprint (none) -> Diodes_SMD:SMA_Handsoldering
- IC1: footprint DIP6 -> Sockets_DIP:DIP-6__300_ELL
- IC2, IC3, IC4: footprint (none) -> sven:8-MSOP
- IC5: footprint TQFP32 -> Housings_QFP:TQFP-32_7x7mm_Pitch0.8mm
- P1, P2: footprint (none) -> Socket_Strips:Socket_Strip_Straight_1x03
- P3: footprint (none) -> Socket_Strips:Socket_Strip_Straight_1x02
- P4: renamed from P?; footprint (none) -> Socket_Strips:Socket_Strip_Straight_2x02
- Q1, Q10, Q11, Q12, Q2, Q3, Q4, Q5, Q6, Q7, Q8, Q9: footprint (none) -> toni:SO8_WITH_EP
- R1, R11, R12, R13, R14, R15, R16, R17, R2, R3, R4, R5, R6, R7, R8, R9: footprint (none) -> Resistors_SMD:R_0805_HandSoldering
- U1: footprint ~ -> toni:SOT223_GND_VO_VI
- U2: renamed from U?; footprint ~ -> toni:SOT223_GND_VO_VI
- Y1: footprint (none) -> toni:CerOsc_3,2x1,3

Commit message: PCB weiter+Layout R
Parts:
- added R10, R18, R19, R20, R21, R22: R, Resistors_SMD:R_0603_HandSoldering, symbol R
- C14, C15, C16: footprint Capacitors_SMD:C_0805_HandSoldering -> Capacitors_SMD:C_0603_HandSoldering
- Q1, Q10, Q11, Q12, Q2, Q3, Q4, Q5, Q6, Q7, Q8, Q9: footprint toni:SO8_WITH_EP -> sven:SO8_WITH_Heatpipes
- R11, R12, R13, R14, R15, R3, R4, R5, R8, R9: footprint Resistors_SMD:R_0805_HandSoldering -> Resistors_SMD:R_0603_HandSoldering
Connections:
- net A_Highside_Gate: now also R10.1; no longer IC2.3 (HO)
- net A_Lowside_Gate: now also R18.1; no longer IC2.8 (LO)
- net B_Highside_Gate: now also R19.1; no longer IC3.3 (HO)
- net B_Lowside_Gate: now also R20.1; no longer IC3.8 (LO)
- net C_Highside_Gate: now also R21.1; no longer IC4.3 (HO)
- net C_Lowside_Gate: now also R22.1; no longer IC4.8 (LO)
- new net: IC2.3 (HO), R10.2
- new net: IC2.8 (LO), R18.2
- new net: IC3.3 (HO), R19.2
- new net: IC3.8 (LO), R20.2
- new net: IC4.3 (HO), R21.2
- new net: IC4.8 (LO), R22.2
Changed lines of the file:
@@
 F 0 "C14" H 5650 9150 40  0000 L CNN
 F 1 "100n" H 5656 8965 40  0000 L CNN
-F 2 "Capacitors_SMD:C_0805_HandSoldering" H 5688 8900 30  0001 C CNN
+F 2 "Capacitors_SMD:C_0603_HandSoldering" H 5688 8900 30  0001 C CNN
 F 3 "" H 5650 9050 60  0000 C CNN
 	1    5650 9050
@@
 F 0 "C15" H 5900 9150 40  0000 L CNN
 F 1 "100n" H 5906 8965 40  0000 L CNN
-F 2 "Capacitors_SMD:C_0805_HandSoldering" H 5938 8900 30  0001 C CNN
+F 2 "Capacitors_SMD:C_0603_HandSoldering" H 5938 8900 30  0001 C CNN
 F 3 "" H 5900 9050 60  0000 C CNN
 	1    5900 9050
@@
 F 0 "C16" H 6150 9150 40  0000 L CNN
 F 1 "100n" H 6156 8965 40  0000 L CNN
-F 2 "Capacitors_SMD:C_0805_HandSoldering" H 6188 8900 30  0001 C CNN
+F 2 "Capacitors_SMD:C_0603_HandSoldering" H 6188 8900 30  0001 C CNN
 F 3 "" H 6150 9050 60  0000 C CNN
 	1    6150 9050
@@
 F 0 "R12" V 1530 8200 40  0000 C CNN
 F 1 "100" V 1457 8201 40  0000 C CNN
-F 2 "Resistors_SMD:R_0805_HandSoldering" V 1380 8200 30  0001 C CNN
+F 2 "Resistors_SMD:R_0603_HandSoldering" V 1380 8200 30  0001 C CNN
 F 3 "" H 1450 8200 30  0000 C CNN
 	1    1450 8200
@@
 F 0 "Q4" H 14210 3070 60  0000 R CNN
 F 1 "MOSFET_N" H 14210 2750 60  0000 R CNN
-F 2 "toni:SO8_WITH_EP" H 14200 2900 60  0001 C CNN
+F 2 "sven:SO8_WITH_Heatpipes" H 14200 2900 60  0001 C CNN
 F 3 "" H 14200 2900 60  0000 C CNN
 	1    14200 2900
@@
 F 0 "R4" V 10780 2700 40  0000 C CNN
 F 1 "18k" V 10707 2701 40  0000 C CNN
-F 2 "Resistors_SMD:R_0805_HandSoldering" V 10630 2700 30  0001 C CNN
+F 2 "Resistors_SMD:R_0603_HandSoldering" V 10630 2700 30  0001 C CNN
 F 3 "" H 10700 2700 30  0000 C CNN
 	1    10700 2700
@@
 F 0 "R5" V 10430 3250 40  0000 C CNN
 F 1 "3k3" V 10357 3251 40  0000 C CNN
-F 2 "Resistors_SMD:R_0805_HandSoldering" V 10280 3250 30  0001 C CNN
+F 2 "Resistors_SMD:R_0603_HandSoldering" V 10280 3250 30  0001 C CNN
 F 3 "" H 10350 3250 30  0000 C CNN
 	1    10350 3250
@@
 F 0 "R3" V 10080 2700 40  0000 C CNN
 F 1 "3k3" V 10007 2701 40  0000 C CNN
-F 2 "Resistors_SMD:R_0805_HandSoldering" V 9930 2700 30  0001 C CNN
+F 2 "Resistors_SMD:R_0603_HandSoldering" V 9930 2700 30  0001 C CNN
 F 3 "" H 10000 2700 30  0000 C CNN
 	1    10000 2700
@@
 F 0 "Q3" H 13460 3070 60  0000 R CNN
 F 1 "MOSFET_N" H 13460 2750 60  0000 R CNN
-F 2 "toni:SO8_WITH_EP" H 13450 2900 60  0001 C CNN
+F 2 "sven:SO8_WITH_Heatpipes" H 13450 2900 60  0001 C CNN
 F 3 "" H 13450 2900 60  0000 C CNN
 	1    13450 2900
@@
 Text GLabel 10950 2700 2    60   Output ~ 0
 A
-Wire Wire Line
-	12700 2500 13050 2500
-Wire Wire Line
-	13050 2500 13050 2300
-Wire Wire Line
-	13050 2300 14000 2300
-Wire Wire Line
-	12950 2900 14000 2900
-Wire Wire Line
-	12950 2900 12950 3000
-Wire Wire Line
-	12950 3000 12700 3000
 Connection ~ 13250 2900
 Wire Wire Line
@@
 F 0 "Q2" H 14210 2470 60  0000 R CNN
 F 1 "MOSFET_N" H 14210 2150 60  0000 R CNN
-F 2 "toni:SO8_WITH_EP" H 14200 2300 60  0001 C CNN
+F 2 "sven:SO8_WITH_Heatpipes" H 14200 2300 60  0001 C CNN
 F 3 "" H 14200 2300 60  0000 C CNN
 	1    14200 2300
@@
 F 0 "Q1" H 13460 2470 60  0000 R CNN
 F 1 "MOSFET_N" H 13460 2150 60  0000 R CNN
-F 2 "toni:SO8_WITH_EP" H 13450 2300 60  0001 C CNN
+F 2 "sven:SO8_WITH_Heatpipes" H 13450 2300 60  0001 C CNN
 F 3 "" H 13450 2300 60  0000 C CNN
 	1    13450 2300
@@
 F 0 "Q8" H 14210 5720 60  0000 R CNN
 F 1 "MOSFET_N" H 14210 5400 60  0000 R CNN
-F 2 "toni:SO8_WITH_EP" H 14200 5550 60  0001 C CNN
+F 2 "sven:SO8_WITH_Heatpipes" H 14200 5550 60  0001 C CNN
 F 3 "" H 14200 5550 60  0000 C CNN
 	1    14200 5550
@@
 F 0 "R9" V 10780 5350 40  0000 C CNN
 F 1 "18k" V 10707 5351 40  0000 C CNN
-F 2 "Resistors_SMD:R_0805_HandSoldering" V 10630 5350 30  0001 C CNN
+F 2 "Resistors_SMD:R_0603_HandSoldering" V 10630 5350 30  0001 C CNN
 F 3 "" H 10700 5350 30  0000 C CNN
 	1    10700 5350
@@
 F 0 "R11" V 10430 5900 40  0000 C CNN
 F 1 "3k3" V 10357 5901 40  0000 C CNN
-F 2 "Resistors_SMD:R_0805_HandSoldering" V 10280 5900 30  0001 C CNN
+F 2 "Resistors_SMD:R_0603_HandSoldering" V 10280 5900 30  0001 C CNN
 F 3 "" H 10350 5900 30  0000 C CNN
 	1    10350 5900
@@
 F 0 "R8" V 10080 5350 40  0000 C CNN
 F 1 "3k3" V 10007 5351 40  0000 C CNN
-F 2 "Resistors_SMD:R_0805_HandSoldering" V 9930 5350 30  0001 C CNN
+F 2 "Resistors_SMD:R_0603_HandSoldering" V 9930 5350 30  0001 C CNN
 F 3 "" H 10000 5350 30  0000 C CNN
 	1    10000 5350
@@
 F 0 "Q7" H 13460 5720 60  0000 R CNN
 F 1 "MOSFET_N" H 13460 5400 60  0000 R CNN
-F 2 "toni:SO8_WITH_EP" H 13450 5550 60  0001 C CNN
+F 2 "sven:SO8_WITH_Heatpipes" H 13450 5550 60  0001 C CNN
 F 3 "" H 13450 5550 60  0000 C CNN
 	1    13450 5550
@@
 Text GLabel 10950 5350 2    60   Output ~ 0
 B
-Wire Wire Line
-	12700 5150 13050 5150
-Wire Wire Line
-	13050 5150 13050 4950
-Wire Wire Line
-	13050 4950 14000 4950
-Wire Wire Line
-	12950 5550 14000 5550
-Wire Wire Line
-	12950 5550 12950 5650
-Wire Wire Line
-	12950 5650 12700 5650
 Connection ~ 13250 5550
 Wire Wire Line
@@
 F 0 "Q6" H 14210 5120 60  0000 R CNN
 F 1 "MOSFET_N" H 14210 4800 60  0000 R CNN
-F 2 "toni:SO8_WITH_EP" H 14200 4950 60  0001 C CNN
+F 2 "sven:SO8_WITH_Heatpipes" H 14200 4950 60  0001 C CNN
 F 3 "" H 14200 4950 60  0000 C CNN
 	1    14200 4950
@@
 F 0 "Q5" H 13460 5120 60  0000 R CNN
 F 1 "MOSFET_N" H 13460 4800 60  0000 R CNN
-F 2 "toni:SO8_WITH_EP" H 13450 4950 60  0001 C CNN
+F 2 "sven:SO8_WITH_Heatpipes" H 13450 4950 60  0001 C CNN
 F 3 "" H 13450 4950 60  0000 C CNN
 	1    13450 4950
@@
 F 0 "Q12" H 14210 8620 60  0000 R CNN
 F 1 "MOSFET_N" H 14210 8300 60  0000 R CNN
-F 2 "toni:SO8_WITH_EP" H 14200 8450 60  0001 C CNN
+F 2 "sven:SO8_WITH_Heatpipes" H 14200 8450 60  0001 C CNN
 F 3 "" H 14200 8450 60  0000 C CNN
 	1    14200 8450
@@
 F 0 "R14" V 10780 8250 40  0000 C CNN
 F 1 "18k" V 10707 8251 40  0000 C CNN
-F 2 "Resistors_SMD:R_0805_HandSoldering" V 10630 8250 30  0001 C CNN
+F 2 "Resistors_SMD:R_0603_HandSoldering" V 10630 8250 30  0001 C CNN
 F 3 "" H 10700 8250 30  0000 C CNN
 	1    10700 8250
@@
 F 0 "R15" V 10430 8800 40  0000 C CNN
 F 1 "3k3" V 10357 8801 40  0000 C CNN
-F 2 "Resistors_SMD:R_0805_HandSoldering" V 10280 8800 30  0001 C CNN
+F 2 "Resistors_SMD:R_0603_HandSoldering" V 10280 8800 30  0001 C CNN
 F 3 "" H 10350 8800 30  0000 C CNN
 	1    10350 8800
@@
 F 0 "R13" V 10080 8250 40  0000 C CNN
 F 1 "3k3" V 10007 8251 40  0000 C CNN
-F 2 "Resistors_SMD:R_0805_HandSoldering" V 9930 8250 30  0001 C CNN
+F 2 "Resistors_SMD:R_0603_HandSoldering" V 9930 8250 30  0001 C CNN
 F 3 "" H 10000 8250 30  0000 C CNN
 	1    10000 8250
@@
 F 0 "Q11" H 13460 8620 60  0000 R CNN
 F 1 "MOSFET_N" H 13460 8300 60  0000 R CNN
-F 2 "toni:SO8_WITH_EP" H 13450 8450 60  0001 C CNN
+F 2 "sven:SO8_WITH_Heatpipes" H 13450 8450 60  0001 C CNN
 F 3 "" H 13450 8450 60  0000 C CNN
 	1    13450 8450
@@
 Text GLabel 10950 8250 2    60   Output ~ 0
 C
-Wire Wire Line
-	12700 8050 13050 8050
-Wire Wire Line
-	13050 8050 13050 7850
-Wire Wire Line
-	13050 7850 14000 7850
-Wire Wire Line
-	12950 8450 14000 8450
-Wire Wire Line
-	12950 8450 12950 8550
-Wire Wire Line
-	12950 8550 12700 8550
 Connection ~ 13250 8450
 Wire Wire Line
@@
 F 0 "Q10" H 14210 8020 60  0000 R CNN
 F 1 "MOSFET_N" H 14210 7700 60  0000 R CNN
-F 2 "toni:SO8_WITH_EP" H 14200 7850 60  0001 C CNN
+F 2 "sven:SO8_WITH_Heatpipes" H 14200 7850 60  0001 C CNN
 F 3 "" H 14200 7850 60  0000 C CNN
 	1    14200 7850
@@
 F 0 "Q9" H 13460 8020 60  0000 R CNN
 F 1 "MOSFET_N" H 13460 7700 60  0000 R CNN
-F 2 "toni:SO8_WITH_EP" H 13450 7850 60  0001 C CNN
+F 2 "sven:SO8_WITH_Heatpipes" H 13450 7850 60  0001 C CNN
 F 3 "" H 13450 7850 60  0000 C CNN
 	1    13450 7850
@@
 Text Label 2000 6300 0    60   ~ 0
 VBat_to_10V
+$Comp
+L R R21
+U 1 1 564B1277
+P 12950 8050
+F 0 "R21" V 13030 8050 40  0000 C CNN
+F 1 "R" V 12957 8051 40  0000 C CNN
+F 2 "Resistors_SMD:R_0603_HandSoldering" V 12880 8050 30  0001 C CNN
+F 3 "" H 12950 8050 30  0000 C CNN
+	1    12950 8050
+	0    1    1    0
+$EndComp
+$Comp
+L R R22
+U 1 1 564B1464
+P 12950 8550
+F 0 "R22" V 13030 8550 40  0000 C CNN
+F 1 "R" V 12957 8551 40  0000 C CNN
+F 2 "Resistors_SMD:R_0603_HandSoldering" V 12880 8550 30  0001 C CNN
+F 3 "" H 12950 8550 30  0000 C CNN
+	1    12950 8550
+	0    1    1    0
+$EndComp
+Wire Wire Line
+	13200 8550 13200 8450
+Wire Wire Line
+	13200 8450 14000 8450
+Wire Wire Line
+	13250 7850 14000 7850
+Wire Wire Line
+	13250 7850 13250 8050
+Wire Wire Line
+	13250 8050 13200 8050
+$Comp
+L R R20
+U 1 1 564B1C36
+P 12950 5650
+F 0 "R20" V 13030 5650 40  0000 C CNN
+F 1 "R" V 12957 5651 40  0000 C CNN
+F 2 "Resistors_SMD:R_0603_HandSoldering" V 12880 5650 30  0001 C CNN
+F 3 "" H 12950 5650 30  0000 C CNN
+	1    12950 5650
+	0    1    1    0
+$EndComp
+$Comp
+L R R19
+U 1 1 564B1E68
+P 12950 5150
+F 0 "R19" V 13030 5150 40  0000 C CNN
+F 1 "R" V 12957 5151 40  0000 C CNN
+F 2 "Resistors_SMD:R_0603_HandSoldering" V 12880 5150 30  0001 C CNN
+F 3 "" H 12950 5150 30  0000 C CNN
+	1    12950 5150
+	0    1    1    0
+$EndComp
+Wire Wire Line
+	13200 5150 13200 4950
+Wire Wire Line
+	13200 4950 14000 4950
+Wire Wire Line
+	13250 5550 14000 5550
+Wire Wire Line
+	13250 5550 13250 5650
+Wire Wire Line
+	13250 5650 13200 5650
+$Comp
+L R R18
+U 1 1 564B272A
+P 12950 3000
+F 0 "R18" V 13030 3000 40  0000 C CNN
+F 1 "R" V 12957 3001 40  0000 C CNN
+F 2 "Resistors_SMD:R_0603_HandSoldering" V 12880 3000 30  0001 C CNN
+F 3 "" H 12950 3000 30  0000 C CNN
+	1    12950 3000
+	0    1    1    0
+$EndComp
+$Comp
+L R R10
+U 1 1 564B287A
+P 12950 2500
+F 0 "R10" V 13030 2500 40  0000 C CNN
+F 1 "R" V 12957 2501 40  0000 C CNN
+F 2 "Resistors_SMD:R_0603_HandSoldering" V 12880 2500 30  0001 C CNN
+F 3 "" H 12950 2500 30  0000 C CNN
+	1    12950 2500
+	0    1    1    0
+$EndComp
+Wire Wire Line
+	13200 3000 13200 2900
+Wire Wire Line
+	13200 2900 14000 2900
+Wire Wire Line
+	13200 2300 14000 2300
+Wire Wire Line
+	13200 2300 13200 2500
 $EndSCHEMATC

Commit message: PCB almost done!
Parts:
- C10, C12, C13, C14, C15, C16, C17, C18, C4, C5, C7: symbol C -> C-RESCUE-esc
- IC1: symbol 4N25 -> 4N25-RESCUE-esc
- R1, R10, R11, R12, R13, R14, R15, R17, R18, R19, R2, R20, R21, R22, R3, R4, R5, R6, R8, R9: symbol R -> R-RESCUE-esc
- R16, R7: footprint Resistors_SMD:R_0805_HandSoldering -> Resistors_SMD:R_0603_HandSoldering; symbol R -> R-RESCUE-esc

Commit message: PCB V1.0
Parts:
- added P5, P6: CONN_01X01, Connect:1pin, symbol CONN_01X01
Connections:
- net GND: now also P5.1 (P1), P6.1 (P1)
Changed lines of the file:
@@
 Wire Wire Line
 	13200 2300 13200 2500
+$Comp
+L CONN_01X01 P5
+U 1 1 564C4523
+P 4500 1900
+F 0 "P5" H 4500 2000 50  0000 C CNN
+F 1 "CONN_01X01" V 4600 1900 50  0000 C CNN
+F 2 "Connect:1pin" H 4500 1900 60  0001 C CNN
+F 3 "" H 4500 1900 60  0000 C CNN
+	1    4500 1900
+	0    -1   -1   0
+$EndComp
+$Comp
+L CONN_01X01 P6
+U 1 1 564C47FE
+P 4700 1900
+F 0 "P6" H 4700 2000 50  0000 C CNN
+F 1 "CONN_01X01" V 4800 1900 50  0000 C CNN
+F 2 "Connect:1pin" H 4700 1900 60  0001 C CNN
+F 3 "" H 4700 1900 60  0000 C CNN
+	1    4700 1900
+	0    -1   -1   0
+$EndComp
+$Comp
+L GND-RESCUE-esc #PWR047
+U 1 1 564C48DB
+P 4500 2100
+F 0 "#PWR047" H 4500 2100 30  0001 C CNN
+F 1 "GND" H 4500 2030 30  0001 C CNN
+F 2 "" H 4500 2100 60  0000 C CNN
+F 3 "" H 4500 2100 60  0000 C CNN
+	1    4500 2100
+	1    0    0    -1
+$EndComp
+$Comp
+L GND-RESCUE-esc #PWR048
+U 1 1 564C49AF
+P 4700 2100
+F 0 "#PWR048" H 4700 2100 30  0001 C CNN
+F 1 "GND" H 4700 2030 30  0001 C CNN
+F 2 "" H 4700 2100 60  0000 C CNN
+F 3 "" H 4700 2100 60  0000 C CNN
+	1    4700 2100
+	1    0    0    -1
+$EndComp
 $EndSCHEMATC
