File: esc.kicad_pcb (KiCad board)
At the start: 2 copper layers, 50 x 60.5 mm, 79 parts, among them IC2 LM25101, IC3 LM25101, IC4 LM25101, IC5 ATMEGA8-AI, P1 CONN_01X03, P2 CONN_01X03, P3 CONN_01X02, P4 CONN_02X02, P5 CONN_01X01, P6 CONN_01X01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

Commit message: Versionierung geändert
Other:
- board text added: "Sven T. S. Rev:1.1"
- board text removed: "Sven T. S. Rev:1"
- board text removed: "Toni Bratsch"
Changed lines of the file:
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@@
-(kicad_pcb (version 4) (host pcbnew 0.201511171411+6319~30~ubuntu15.10.1-product)
+(kicad_pcb (version 4) (host pcbnew 0.201512031508+6343~38~ubuntu15.10.1-stable)
   (general
     (links 436)
@@
     )
   )
-  (gr_text "Toni Bratsch" (at 212.852 109.347) (layer F.SilkS)
+  (gr_text "Toni Bartsch" (at 212.852 109.347) (layer F.SilkS)
     (effects (font (size 1 1) (thickness 0.1)))
   )
@@
     (effects (font (size 1.5 1.5) (thickness 0.3)))
   )
-  (gr_text "Sven T. S. Rev:1" (at 219.456 109.474) (layer B.Cu)
+  (gr_text "Sven T. S. Rev:1.1\n" (at 218.948 109.474) (layer B.Cu)
     (effects (font (size 1.5 1.5) (thickness 0.3)) (justify mirror))
   )
